File: Hardware/schematic.kicad_sch (KiCad schematic)
At the start: 4 parts, among them U1 ESP32-WROOM-32E, U2 HX711, U3 MPU-6050, U4 MAX30102

Commit message: feat:pushed the main
Connections:
- net at U3.1 (CLKIN): now also U1.3 (EN)
- net at U3.10 (REGOUT): now also U1.10 (IO25), U1.11 (IO26), U3.20 (CPOUT)
- net at U3.12 (INT): now also U1.29 (IO5)
- net GND: now reaches U3.13 (VDD)
- net GND: now also U3.18 (GND), U4.13 (~{INT})
- net at U3.23 (SCL): now also U1.35 (TXD0/IO1)
- net at U3.24 (SDA): now also U1.25 (IO0)
- net at U2.12 (DOUT): now also U1.8 (IO32)
- net at U2.13 (XO): now also U1.6 (IO34)
- net at U2.14 (XI): now also U1.9 (IO33)
- net at U2.2 (BASE): now also U1.16 (IO13), U2.3 (AVDD)
- net at U4.11 (VDD): now also U1.7 (IO35)
- net at U4.12 (GND): now also U1.34 (RXD0/IO3), U4.3 (SDA), U4.4 (PGND)
- net at U4.2 (SCL): now also U1.24 (IO2)
