File: Hardware/_restore_backup_2026-08-27T15-58-32-780/schematic.kicad_sch (KiCad schematic)
At the start: 5 parts, among them U1 ESP32-WROOM-32E, U2 HX711, U3 MPU-6050, U4 MAX30102

Commit message: feat: restructuring files for the project
Parts:
- removed A1: Arduino_Nano_v3.x, Module:Arduino_Nano, symbol MCU_Module:Arduino_Nano_v3.x
Connections:
- net at U2.2 (BASE): now also U2.3 (AVDD)
Other:
- moved on the sheet: U2
Changed lines of the file:
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@@
 	(generator_version "10.0")
 	(paper "A4")
+	(junction
+		(at 170.18 77.47)
+		(diameter 0)
+		(color 0 0 0 0)
+	)
+	(wire
+		(pts
+			(xy 170.18 77.47) (xy 170.18 78.74)
+		)
+		(stroke
+			(width 0)
+			(type default)
+		)
+	)
+	(wire
+		(pts
+			(xy 167.64 104.14) (xy 157.48 104.14)
+		)
+		(stroke
+			(width 0)
+			(type default)
+		)
+	)
+	(wire
+		(pts
+			(xy 170.18 74.93) (xy 170.18 77.47)
+		)
+		(stroke
+			(width 0)
+			(type default)
+		)
+	)
+	(wire
+		(pts
+			(xy 157.48 106.68) (xy 166.37 106.68)
+		)
+		(stroke
+			(width 0)
+			(type default)
+		)
+	)
+	(wire
+		(pts
+			(xy 170.18 88.9) (xy 170.18 87.63)
+		)
+		(stroke
+			(width 0)
+			(type default)
+		)
+	)
 	(symbol
 		(lib_id "Sensor_Motion:MPU-6050")
@@
 	(symbol
 		(lib_id "Analog_ADC:HX711")
-		(at 195.58 81.28 0)
+		(at 182.88 87.63 0)
 		(unit 1)
 		(body_style 1)
@@
 		(fields_autoplaced yes)
 		(property "Reference" "U2"
-			(at 197.7233 101.6 0)
+			(at 185.0233 107.95 0)
 			(show_name no)
 			(do_not_autoplace no)
@@
 		)
 		(property "Value" "HX711"
-			(at 197.7233 104.14 0)
+			(at 185.0233 110.49 0)
 			(show_name no)
 			(do_not_autoplace no)
@@
 		)
 		(property "Footprint" "Package_SO:SOIC-16_3.9x9.9mm_P1.27mm"
-			(at 199.39 80.01 0)
+			(at 186.69 86.36 0)
 			(hide yes)
 			(show_name no)
@@
 		)
 		(property "Datasheet" "https://web.archive.org/web/20220615044707/https://akizukidenshi.com/download/ds/avia/hx711.pdf"
-			(at 199.39 82.55 0)
+			(at 186.69 88.9 0)
 			(hide yes)
 			(show_name no)
@@
 		)
 		(property "Description" "24-bit Analog-to-Digital Converter (ADC) for Weight Scales, SOIC-16 (SOP-16)"
-			(at 195.58 81.28 0)
+			(at 182.88 87.63 0)
 			(hide yes)
 			(show_name no)
@@
 					(unit 1)
 				)
-			)
-		)
-	)
-	(symbol
-		(lib_id "MCU_Module:Arduino_Nano_v3.x")
-		(at 101.6 46.99 0)
-		(unit 1)
-		(body_style 1)
-		(exclude_from_sim no)
-		(in_bom yes)
-		(on_board yes)
-		(in_pos_files yes)
-		(dnp no)
-		(fields_autoplaced yes)
-		(property "Reference" "A1"
-			(at 106.2833 72.39 0)
-			(show_name no)
-			(do_not_autoplace no)
-			(effects
-				(font
-					(size 1.27 1.27)
-				)
-				(justify left)
-			)
-		)
-		(property "Value" "Arduino_Nano_v3.x"
-			(at 106.2833 74.93 0)
-			(show_name no)
-			(do_not_autoplace no)
-			(effects
-				(font
-					(size 1.27 1.27)
-				)
-				(justify left)
-			)
-		)
-		(property "Footprint" "Module:Arduino_Nano"
-			(at 101.6 46.99 0)
-			(hide yes)
-			(show_name no)
-			(do_not_autoplace no)
-			(effects
-				(font
-					(size 1.27 1.27)
-					(italic yes)
-				)
-			)
-		)
-		(property "Datasheet" "http://www.mouser.com/pdfdocs/Gravitech_Arduino_Nano3_0.pdf"
-			(at 101.6 46.99 0)
-			(hide yes)
-			(show_name no)
-			(do_not_autoplace no)
-			(effects
-				(font
-					(size 1.27 1.27)
-				)
-			)
-		)
-		(property "Description" "Arduino Nano v3.x"
-			(at 101.6 46.99 0)
-			(hide yes)
-			(show_name no)
-			(do_not_autoplace no)
-			(effects
-				(font
-					(size 1.27 1.27)
-				)
-			)
-		)
-		(pin "19"
-		)
-		(pin "23"
-		)
-		(pin "9"
-		)
-		(pin "20"
-		)
-		(pin "17"
-		)
-		(pin "22"
-		)
-		(pin "29"
-		)
-		(pin "1"
-		)
-		(pin "3"
-		)
-		(pin "7"
-		)
-		(pin "2"
-		)
-		(pin "6"
-		)
-		(pin "11"
-		)
-		(pin "4"
-		)
-		(pin "10"
-		)
-		(pin "12"
-		)
-		(pin "13"
-		)
-		(pin "14"
-		)
-		(pin "15"
-		)
-		(pin "8"
-		)
-		(pin "16"
-		)
-		(pin "18"
-		)
-		(pin "5"
-		)
-		(pin "21"
-		)
-		(pin "24"
-		)
-		(pin "25"
-		)
-		(pin "26"
-		)
-		(pin "27"
-		)
-		(pin "28"
-		)
-		(pin "30"
-		)
-		(instances
-			(project "schematic"
-				(path "/62d25dba-bbf5-4c29-afa2-e2397d4820c7"
-					(reference "A1")
-					(unit 1)
-				)
